File: pcb/ad9866_2.kicad_pcb (KiCad board)
At the start: 4 copper layers, 50 x 50 mm, 103 parts, among them CN1 MEC6-140_CONNECTOR_BEMICRO, CON1 USB-MICRO-B, P1 CONN_2, P10 CONN_1, P2 CONN_10X2, P3 CONN_1, P4 CONN_5X2, P5 CONN_1, P5V0 CONN_1, P6 Coaxial_Connector, P7 Coaxial_Connector, P8 CONN_2, P9 CONN_1, Q1 Si2301, T1 TRANSF_ADT2, T2 TRANSF_ADT8, U1 NCP1117ST33T3G, U2 NCP1117ST33T3G, U3 Si510, U4 AD9866BCPZ, U5 NCP1117ST33T3G, U6 25AA02E48T-I/OT

Commit message: ground plane revisions
Parts:
- PDVDD1: moved to F.Cu
Routing:
- net Net-(C6-Pad1): vias 0 -> 1

Commit message: Revised after first review.
Parts:
- removed PGND1: CONN_1, Measurement_Points:Measurement_Point_Round-SMD-Pad_Small
- added C11: 0.1UF, Capacitors_SMD:c_0805, F.Cu at (171.6, 48.4)
- added C13: 0.1UF, Capacitors_SMD:c_0805, F.Cu at (171.4, 61.4)
- added FB35: FB, SMD_Packages:SM0805, F.Cu at (170.5, 51.1)
- C10, C12, C14, C18, C19, C24, C32, C35, C8, D1, P7, R2, T2: moved to B.Cu
- moved T2 10.5 mm to (159.6, 75.2), turned to 180 degrees
- moved C9 7.46 mm to (164.4, 50.0)
- moved C14 7.18 mm to (165.5, 53.9)
- moved C12 6.45 mm to (165.5, 56.2), turned to 0 degrees
- moved P5 6.33 mm to (142.1, 39.5)
- moved C37 6.33 mm to (165.5, 59.6), turned to 270 degrees
- moved R1 6.25 mm to (162.7, 65.0)
- moved C8 5.75 mm to (157.6, 53.9), turned to 180 degrees
- moved C17 5.58 mm to (157.1, 65.7), turned to 270 degrees
- moved C16 5.40 mm to (156.8, 59.4), turned to 270 degrees
- moved P10 4.89 mm to (163.9, 68.6)
- moved P9 4.83 mm to (168.6, 68.5)
- moved C32 4.61 mm to (152.2, 76.7), turned to 0 degrees
- moved C24 3.96 mm to (161.7, 59.6), turned to 270 degrees
- moved R2 3.74 mm to (151.6, 54.0)
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Connections:
- CN1 pad 79: VIN -> Net-(C11-Pad2)
- CN1 pad 80: VIN -> Net-(C11-Pad2)
- T2 pad 1: Net-(C32-Pad1) -> GND
- T2 pad 3: GND -> Net-(C32-Pad1)
- T2 pad 4: Net-(C19-Pad1) -> Net-(C18-Pad1)
- T2 pad 6: Net-(C18-Pad1) -> Net-(C19-Pad1)
Routing:
- net GND: track 510.3 -> 152.3 mm, vias 35 -> 84
- net /CLKVDD: track 35.5 -> 67.9 mm, vias 1 -> 3
- net /AVDD_DAC: track 23.9 -> 49.9 mm, vias 1 -> 3
- net Net-(C11-Pad2): track 0.00 -> 14.9 mm
- net Net-(FB23-Pad1): track 28.6 -> 14.8 mm, vias 2 -> 0
- net Net-(P6-Pad1): track 23.6 -> 10.7 mm
- net /P55: track 43.4 -> 55.2 mm
- net Net-(CN1-Pad34): track 24.5 -> 32.6 mm
- net VIN: track 118.0 -> 125.6 mm, vias 1 -> 4
- net Net-(C18-Pad1): track 9.67 -> 2.26 mm
- net Net-(C5-Pad1): track 10.1 -> 17.2 mm
- net /AVDD_ADC: track 29.5 -> 22.6 mm
- net /SEN: track 17.6 -> 23.8 mm
- net /EXP_PR: track 40.3 -> 45.9 mm
- net Net-(R1-Pad2): track 10.0 -> 4.77 mm
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Other:
- net class Default: clearance 0.16 -> 0.155
- net class GND added: clearance 0.155, trace_width 0.3, via_dia 0.4, via_drill 0.3
- net class Power added: clearance 0.155, trace_width 0.3, via_dia 0.4, via_drill 0.3
- rule trace_clearance: 0.16 -> 0.155
- rule trace_min: 0.16 -> 0.1524
- board text added: "Hermes-Lite v 1.1 KL7NA"
- board text removed: "Hermes-Lite v 1.1 KF7O/KL7NA"
